Commit message: Add hardware point cloud calibration pipeline

File: urdf_rc5_right_hand/Robot_with_right_hand_cor_fixed.urdf (robot description, URDF)
Before this commit: robot rc5_aero_hand, 42 links, 41 joints
Links:
- removed link d405_depth_frame
- removed link d405_depth_optical_frame
- removed link right_index_tip_link
- removed link right_middle_tip_link
- removed link right_pinky_tip_link
- removed link right_ring_tip_link
- removed link right_thumb_tip_link
- link right_index_distal_link: geometry collision mesh filename=./aero_hand_meshes/right_index_distal_link.STL; collision mesh filename=./aero_hand_meshes/right_index_tip_link.STL
- link right_middle_distal_link: geometry collision mesh filename=./aero_hand_meshes/right_middle_distal_link.STL; collision mesh filename=./aero_hand_meshes/right_middle_tip_link.STL
- link right_pinky_distal_link: geometry collision mesh filename=./aero_hand_meshes/right_pinky_distal_link.STL; collision mesh filename=./aero_hand_meshes/right_pinky_tip_link.STL
- link right_ring_distal_link: geometry collision mesh filename=./aero_hand_meshes/right_ring_distal_link.STL; collision mesh filename=./aero_hand_meshes/right_ring_tip_link.STL
- link right_thumb_distal_link: geometry collision mesh filename=./aero_hand_meshes/right_thumb_distal_link.STL; collision mesh filename=./aero_hand_meshes/right_thumb_tip_link.STL
Joints:
- removed joint d405_depth_to_d405_depth_optical
- removed joint prehand_cam_to_d405_depth
- removed joint right_index_tip
- removed joint right_middle_tip
- removed joint right_pinky_tip
- removed joint right_ring_tip
- removed joint right_thumb_tip
